Commit message: radius, collision, inertia added

File: robot_description/robot_core.xacro (robot description, xacro)
@@ -1,4 +1,5 @@
 <?xml version="1.0"?>
 <robot xmlns:xacro="http://www.ros.org/wiki/xacro" >
+    <xacro:include filename = "inertial_macros.xacro" />
     <material name="white">
         <color rgba="1 1 1 1" />
@@ -33,4 +34,13 @@
             <material name = "white"/>
         </visual>
+        <collision>
+            <origin xyz = "0.15 0 0.075"/>
+            <geometry>
+                <box size = "0.8 0.3 0.15"/>
+            </geometry>
+        </collision>
+        <xacro:inertial_box mass="0.5" x="0.3" y="0.3" z="0.15">
+            <origin xyz="0.15 0 0.075" rpy="0 0 0"/>
+        </xacro:inertial_box>
     </link>
     <!-- LEFT BACK LINK -->
@@ -44,8 +54,16 @@
         <visual>
             <geometry>
-                <cylinder radius = "0.05" length = "0.04" />
+                <cylinder radius = "0.1" length = "0.04" />
             </geometry>
             <material name = "blue" />
         </visual>
+        <collision>
+            <geometry>
+                <cylinder radius = "0.1" length = "0.04" />
+            </geometry>
+        </collision>
+        <xacro:inertial_cylinder mass="0.1" length="0.04" radius="0.1">
+            <origin xyz="0 0 0" rpy="0 0 0"/>
+        </xacro:inertial_cylinder>
     </link>
     <!-- RIGHT BACK LINK -->
@@ -59,8 +77,16 @@
         <visual>
             <geometry>
-                <cylinder radius = "0.05" length = "0.04" />
+                <cylinder radius = "0.1" length = "0.04" />
             </geometry>
             <material name = "blue" />
         </visual>
+        <collision>
+            <geometry>
+                <cylinder radius = "0.1" length = "0.04" />
+            </geometry>
+        </collision>
+        <xacro:inertial_cylinder mass="0.1" length="0.04" radius="0.1">
+            <origin xyz="0 0 0" rpy="0 0 0"/>
+        </xacro:inertial_cylinder>
     </link>
     <!-- LEFT FRONT LINK -->
@@ -74,8 +100,16 @@
         <visual>
             <geometry>
-                <cylinder radius = "0.05" length = "0.04" />
+                <cylinder radius = "0.1" length = "0.04" />
             </geometry>
             <material name = "blue" />
         </visual>
+        <collision>
+            <geometry>
+                <cylinder radius = "0.1" length = "0.04" />
+            </geometry>
+        </collision>
+        <xacro:inertial_cylinder mass="0.1" length="0.04" radius="0.1">
+            <origin xyz="0 0 0" rpy="0 0 0"/>
+        </xacro:inertial_cylinder>
     </link>
     <!-- RIGHT FRONT LINK -->
@@ -89,8 +123,16 @@
         <visual>
             <geometry>
-                <cylinder radius = "0.05" length = "0.04" />
+                <cylinder radius = "0.1" length = "0.04" />
             </geometry>
             <material name = "blue" />
         </visual>
+        <collision>
+            <geometry>
+                <cylinder radius = "0.1" length = "0.04" />
+            </geometry>
+        </collision>
+        <xacro:inertial_cylinder mass="0.1" length="0.04" radius="0.1">
+            <origin xyz="0 0 0" rpy="0 0 0"/>
+        </xacro:inertial_cylinder>
     </link>
 </robot>
