Commit message: gazebo sim done

File: robot_description/robot.urdf.xacro (robot description, xacro)
@@ -2,3 +2,4 @@
 <robot xmlns:xacro="http://www.ros.org/wiki/xacro"  name="robot">
     <xacro:include filename = "robot_core.xacro" />
+    <xacro:include filename = "robot_gazebo.xacro" />
 </robot>

File: robot_description/robot_core.xacro (robot description, xacro)
@@ -17,5 +17,5 @@
         <color rgba="1 0 0 1"/>
     </material>
-    <!-- BASIC LINK -->
+    <!-- BASIC LINK -->s
     <link name = "base_link">
     </link>

File: robot_description/robot_gazebo.xacro (robot description, xacro)
@@ -1,2 +1,43 @@
 <?xml version="1.0"?>
 <robot xmlns:xacro="http://www.ros.org/wiki/xacro">
+	<gazebo reference="base_link">
+        <material>Gazebo/Green</material>
+    </gazebo>
+    <gazebo reference="chassis">
+        <material>Gazebo/Blue</material>
+        <mu1 value="0.001"/>
+        <mu2 value="0.001"/>
+    </gazebo>
+    <gazebo reference="left_wheel_back">
+        <material>Gazebo/Orange</material>
+        <mu1 value="0.001"/>
+        <mu2 value="0.001"/>
+    </gazebo>
+    <gazebo reference="right_wheel_back">
+        <material>Gazebo/Orange</material>
+    </gazebo>
+    <gazebo reference="left_wheel_front">
+        <material>Gazebo/Orange</material>
+    </gazebo>
+    <gazebo reference="right_wheel_front">
+        <material>Gazebo/Orange</material>
+    </gazebo>
+    <gazebo>
+        <plugin name="diff_drive" filename="libgazebo_ros_diff_drive.so">
+            <!-- Wheel Information -->
+            <left_joint>left_wheel_joint_front</left_joint>
+            <right_joint>right_wheel_joint_front</right_joint>
+            <wheel_separation>0.35</wheel_separation>
+            <wheel_diameter>0.1</wheel_diameter>
+            <!-- Limits -->
+            <max_wheel_torque>200</max_wheel_torque>
+            <max_wheel_acceleration>10.0</max_wheel_acceleration>
+            <!-- Output -->
+            <odometry_frame>odom</odometry_frame>
+            <robot_base_frame>base_link</robot_base_frame>
+            <publish_odom>true</publish_odom>
+            <publish_odom_tf>true</publish_odom_tf>
+            <publish_wheel_tf>true</publish_wheel_tf>
+        </plugin>
+    </gazebo>
+</robot>
