Commit message: add showpath node

File: src/test_bot/src/test_bot.urdf (robot description, URDF)
Before this commit: robot sam_bot, 2 links, 1 joints
Links:
- added link map
Joints:
- added joint map_joint: type fixed, parent map, child base_link, origin xyz=0 0 0 rpy=0 0 0

Commit message: add tf_odom

File: src/test_bot/src/test_bot.urdf (robot description, URDF)
Before this commit: robot sam_bot, 3 links, 2 joints
Links:
- removed link map
- added link imu_link; collision box size=0.1 0.1 0.1; visual box size=0.1 0.1 0.1
Joints:
- removed joint map_joint
- added joint imu_joint: type fixed, parent base_link, child imu_link, origin xyz=0 0 0.01

Commit message: add odom

File: src/test_bot/src/test_bot.urdf (robot description, URDF)
Before this commit: robot sam_bot, 3 links, 2 joints
Links:
- added link map
- added link odom
Joints:
- added joint map_joint: type fixed, parent base_link, child map, origin xyz=0 0 0 rpy=0 0 0
- added joint odom_joint: type fixed, parent odom, child base_link, origin xyz=0 0 0 rpy=0 0 0

Commit message: add odom

File: src/test_bot/src/test_bot.urdf (robot description, URDF)
Before this commit: robot sam_bot, 5 links, 4 joints
Links:
- removed link map
Joints:
- removed joint map_joint
